File: The65.kicad_sch (KiCad schematic)
At the start: 166 parts, among them J1 JST_SH, U1 XC6206P332MR-G, U2 STM32F072CBTx

Commit message: fixed columns and rows
the net label on the pcb were wrong. i noticed so when making the firmware for the board
Connections:
- net COL0: now also MX1.1, MX17.1, MX32.1, MX46.1, MX60.1, MXb32.1, MXb60.1, U2.20 (PB2); no longer D1.1 (K), D10.1 (K), D11.1 (K), D12.1 (K), D13.1 (K), D14.1 (K), D15.1 (K), D16.1 (K), D3.1 (K), D4.1 (K), D5.1 (K), D6.1 (K), D7.1 (K), D8.1 (K), D9.1 (K), U2.22 (PB11)
- net COL1: now also MX18.1, MX2.1, MX3.1, MX33.1, MX61.1, MXb61.1, U2.28 (PB15); no longer D17.1 (K), D18.1 (K), D19.1 (K), D20.1 (K), D21.1 (K), D22.1 (K), D23.1 (K), D24.1 (K), D25.1 (K), D26.1 (K), D27.1 (K), D28.1 (K), D29.1 (K), D30.1 (K), D31.1 (K), U2.21 (PB10)
- net COL2: now also MX19.1, MX34.1, MX4.1, MX47.1, MX62.1, MXb62.1, U2.29 (PA8); no longer D32.1 (K), D33.1 (K), D34.1 (K), D35.1 (K), D36.1 (K), D37.1 (K), D38.1 (K), D39.1 (K), D40.1 (K), D41.1 (K), D42.1 (K), D43.1 (K), D44.1 (K), D45.1 (K), U2.12 (PA2)
- net COL3: now also MX20.1, MX35.1, MX48.1, MX5.1, U2.34 (PA13); no longer D2.1 (K), D46.1 (K), D47.1 (K), D48.1 (K), D49.1 (K), D50.1 (K), D51.1 (K), D52.1 (K), D53.1 (K), D54.1 (K), D55.1 (K), D56.1 (K), D57.1 (K), D58.1 (K), D59.1 (K), U2.10 (PA0)
- net COL4: now also MX21.1, MX36.1, MX49.1, MX6.1, U2.31 (PA10); no longer D60.1 (K), D61.1 (K), D62.1 (K), D63.1 (K), D64.1 (K), D65.1 (K), D66.1 (K), D67.1 (K), D68.1 (K), U2.11 (PA1)
- net ROW0: now also D1.1 (K), D10.1 (K), D11.1 (K), D12.1 (K), D13.1 (K), D14.1 (K), D15.1 (K), D16.1 (K), D3.1 (K), D4.1 (K), D5.1 (K), D6.1 (K), D7.1 (K), D8.1 (K), D9.1 (K), U2.22 (PB11); no longer MX1.1, MX17.1, MX32.1, MX46.1, MX60.1, MXb32.1, MXb60.1, U2.20 (PB2)
- net ROW1: now also D17.1 (K), D18.1 (K), D19.1 (K), D20.1 (K), D21.1 (K), D22.1 (K), D23.1 (K), D24.1 (K), D25.1 (K), D26.1 (K), D27.1 (K), D28.1 (K), D29.1 (K), D30.1 (K), D31.1 (K), U2.21 (PB10); no longer MX18.1, MX2.1, MX3.1, MX33.1, MX61.1, MXb61.1, U2.28 (PB15)
- net ROW2: now also D32.1 (K), D33.1 (K), D34.1 (K), D35.1 (K), D36.1 (K), D37.1 (K), D38.1 (K), D39.1 (K), D40.1 (K), D41.1 (K), D42.1 (K), D43.1 (K), D44.1 (K), D45.1 (K), U2.12 (PA2); no longer MX19.1, MX34.1, MX4.1, MX47.1, MX62.1, MXb62.1, U2.29 (PA8)
- net ROW3: now also D2.1 (K), D46.1 (K), D47.1 (K), D48.1 (K), D49.1 (K), D50.1 (K), D51.1 (K), D52.1 (K), D53.1 (K), D54.1 (K), D55.1 (K), D56.1 (K), D57.1 (K), D58.1 (K), D59.1 (K), U2.10 (PA0); no longer MX20.1, MX35.1, MX48.1, MX5.1, U2.34 (PA13)
- net ROW4: now also D60.1 (K), D61.1 (K), D62.1 (K), D63.1 (K), D64.1 (K), D65.1 (K), D66.1 (K), D67.1 (K), D68.1 (K), U2.11 (PA1); no longer MX21.1, MX36.1, MX49.1, MX6.1, U2.31 (PA10)
- net ROW10 renamed COL10
- net ROW11 renamed COL11
- net ROW12 renamed COL12
- net ROW13 renamed COL13
- net ROW14 renamed COL14
- net ROW5 renamed COL5
- net ROW6 renamed COL6
- net ROW7 renamed COL7
- net ROW8 renamed COL8
- net ROW9 renamed COL9
